File: PCB/SHIELD_STM32F426ZI.brd (EAGLE design)
At the start: 73.3 x 110.9 mm, 18 parts, among them Q1 FDN304P, Q2 FDN304P, Q4 SSM3J338R,LF

Commit message: fix route
Parts:
- moved R7 6.49 mm to (50.9, 33.2)
- moved R4 5.46 mm to (45.8, 33.2)
- moved R6 4.05 mm to (49.3, 33.2)
- moved Q2 3.32 mm to (56.7, 32.8)
- moved R5 3.25 mm to (47.6, 33.2)
- moved R8 3.16 mm to (43.8, 33.2)
- moved R9 3.16 mm to (42.2, 33.2)
Connections:
- net CARD_DET: now also STM32F4/F7.CN12_3; no longer STM32F4/F7.CN12_11
- net MOSFET_SDCARD: now also STM32F4/F7.CN11_13; no longer STM32F4/F7.CN11_30
Routing:
- net GND: track 21.3 -> 40.6 mm, vias 4 -> 8
- net MOSFET_SDCARD: track 29.1 -> 20.2 mm, vias 1 -> 0
- net SDIO_D3: track 50.4 -> 41.7 mm, vias 1 -> 0
- net SDIO_D2: track 54.6 -> 46.0 mm, vias 1 -> 0
- net FMC_SDNWE: track 33.3 -> 41.0 mm
- net CARD_DET: track 24.0 -> 31.2 mm, vias 1 -> 0
- net SDIO_CMD: track 46.2 -> 41.8 mm
- net N$1: track 21.3 -> 17.0 mm
- net FMC_SDCLK: track 38.7 -> 34.6 mm
- net SDIO_D0: track 49.0 -> 45.7 mm
- net FMC_SDNRAS: track 47.9 -> 51.1 mm
- net SDIO_CK: track 49.7 -> 46.4 mm, vias 0 -> 1
- net FMC_D0: track 53.6 -> 56.4 mm
- net DCMI_HSYNC: track 89.4 -> 92.0 mm
- net FMC_D15: track 43.1 -> 41.1 mm
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
Commit message: fix route 1
Parts:
- moved C1 9.39 mm to (28.0, 66.8)
- moved CAMERA 9.39 mm to (24.8, 95.1)
- moved PIR 9.39 mm to (51.2, 96.7)
- moved Q1 9.39 mm to (42.9, 96.8)
- moved SDRAM 9.39 mm to (36.7, 73.3)
- moved R2 9.39 mm to (25.5, 42.8)
- moved R4 9.39 mm to (38.5, 27.4)
- moved R5 9.39 mm to (40.2, 27.3)
- moved R6 9.39 mm to (42.0, 27.4)
- moved R8 9.39 mm to (36.4, 27.4)
- moved R9 9.39 mm to (34.9, 27.4)
- moved STM32F4/F7 9.39 mm to (37.5, 52.4)
- moved SDCARD 9.39 mm to (38.2, 5.94)
- moved Q4 9.39 mm to (60.4, 97.2)
- moved R3 9.39 mm to (29.7, 42.8)
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Routing:
- net FMC_SDNE1: track 69.2 -> 75.3 mm, vias 4 -> 3
- net FMC_SDCKE1: track 51.7 -> 55.8 mm
- net FMC_D13: track 70.7 -> 73.9 mm
- net FMC_SDNWE: track 41.0 -> 39.4 mm
- net GND: track 40.6 -> 39.3 mm
- net FMC_A6: track 30.5 -> 29.5 mm
- net FMC_A7: track 27.4 -> 26.6 mm
- net 3.3V: track 169.1 -> 169.8 mm

Commit message: new route 2
Routing:
- net 3.3V: track 169.8 -> 175.9 mm
- net FMC_SDNE1: track 75.3 -> 77.9 mm
- net FMC_SDNRAS: track 51.1 -> 52.1 mm
Other:
- board text added: "3.3V"
- board text added: "D0"
- board text added: "D1"
- board text added: "D2"
- board text added: "D3"
- board text added: "D4"
- board text added: "D5"
- board text added: "D6"
- board text added: "D7"
- board text added: "HSYN"
- board text added: "PIR"
- board text added: "PIXCK"
- board text added: "PWDN"
- board text added: "RESET"
- board text added: "SCL"
- board text added: "SDA"
- board text added: "VSYN"
- board text added: "XCK"

Commit message: new route 3
Parts:
- moved R1 46.2 mm to (32.2, 88.7)
- moved R2 46.1 mm to (28.1, 88.8)
- moved R3 18.3 mm to (28.1, 61.0), turned to 0 degrees
- moved R4 0.05 mm to (38.4, 27.4)
Routing:
- net 3.3V: track 175.9 -> 201.9 mm, vias 11 -> 14
- net DCMI_PIXCK: track 81.9 -> 92.6 mm
- net GND: track 39.3 -> 32.4 mm
- net RESET: track 65.2 -> 70.4 mm
- net RCC_MCO_1: track 67.9 -> 72.0 mm
- net PWDN: track 59.3 -> 61.6 mm
- net FMC_SDNE1: track 77.9 -> 75.8 mm, vias 3 -> 2
- net I2C2_SCL: track 78.6 -> 80.1 mm
- net FMC_D12: track 26.1 -> 25.1 mm
- net I2C2_SDA: track 84.6 -> 84.0 mm, vias 5 -> 2
